Commit message: update code

File: src/vanh_description/urdf/robot_description.urdf (robot description, URDF)
Before this commit: robot orion_urdf, 18 links, 17 joints
Links:
- link back_left_link_1: geometry collision mesh filename=package://vanh_description/meshes/back_left_link_1.STL; visual mesh filename=package://vanh_description/meshes/back_left_link_1.STL
- link back_left_link_2: geometry collision mesh filename=package://vanh_description/meshes/back_left_link_2.STL; visual mesh filename=package://vanh_description/meshes/back_left_link_2.STL
- link back_left_link_3: geometry collision mesh filename=package://vanh_description/meshes/back_left_link_3.STL; visual mesh filename=package://vanh_description/meshes/back_left_link_3.STL
- link back_right_link_1: geometry collision mesh filename=package://vanh_description/meshes/back_right_link_1.STL; visual mesh filename=package://vanh_description/meshes/back_right_link_1.STL
- link back_right_link_2: geometry collision mesh filename=package://vanh_description/meshes/back_right_link_2.STL; visual mesh filename=package://vanh_description/meshes/back_right_link_2.STL
- link back_right_link_3: geometry collision mesh filename=package://vanh_description/meshes/back_right_link_3.STL; visual mesh filename=package://vanh_description/meshes/back_right_link_3.STL
- link chassis_link: geometry collision mesh filename=package://vanh_description/meshes/chassis_link.STL; visual mesh filename=package://vanh_description/meshes/chassis_link.STL
- link front_left_link_1: geometry collision mesh filename=package://vanh_description/meshes/front_left_link_1.STL; visual mesh filename=package://vanh_description/meshes/front_left_link_1.STL
- link front_left_link_2: geometry collision mesh filename=package://vanh_description/meshes/front_left_link_2.STL; visual mesh filename=package://vanh_description/meshes/front_left_link_2.STL
- link front_left_link_3: geometry collision mesh filename=package://vanh_description/meshes/front_left_link_3.STL; visual mesh filename=package://vanh_description/meshes/front_left_link_3.STL
- link front_right_link_1: geometry collision mesh filename=package://vanh_description/meshes/front_right_link_1.STL; visual mesh filename=package://vanh_description/meshes/front_right_link_1.STL
- link front_right_link_2: geometry collision mesh filename=package://vanh_description/meshes/front_right_link_2.STL; visual mesh filename=package://vanh_description/meshes/front_right_link_2.STL
- link front_right_link_3: geometry collision mesh filename=package://vanh_description/meshes/front_right_link_3.STL; visual mesh filename=package://vanh_description/meshes/front_right_link_3.STL
- link laser: geometry collision mesh filename=package://vanh_description/meshes/lidar_link.STL; visual mesh filename=package://vanh_description/meshes/lidar_link.STL
- link left_camera_link: geometry collision mesh filename=package://vanh_description/meshes/left_camera_link.STL; visual mesh filename=package://vanh_description/meshes/left_camera_link.STL
- link lid_link: geometry collision mesh filename=package://vanh_description/meshes/lid_link.STL; visual mesh filename=package://vanh_description/meshes/lid_link.STL
- link right_camera_link: geometry collision mesh filename=package://vanh_description/meshes/right_camera_link.STL; visual mesh filename=package://vanh_description/meshes/right_camera_link.STL
